File: uyLy_LFChassis/uyLy_LFChassis.kicad_pcb (KiCad board)
At the start: 2 copper layers, 98 x 155.8 mm, 24 parts, among them J1 Conn_01x08_Socket, J2 Conn_01x02_Pin, J3 Conn_01x02_Pin, J4 Conn_01x02_Pin, J5 Conn_01x02_Socket, J6 Conn_01x01_Socket, SW1 SW_DIP_x04, U1 TB6612FNG

Commit message: update: pcb design
Parts:
- removed J5: Conn_01x02_Socket, Connector_PinHeader_2.54mm:PinHeader_1x02_P2.54mm_Horizontal
- removed J6: Conn_01x01_Socket, Connector_PinHeader_2.54mm:PinHeader_1x01_P2.54mm_Horizontal
- removed the REF** at (304.6, 183.4)
- removed the REF** at (288.6, 177.4)
- removed the REF** at (304.6, 189.4)
- removed the REF** at (304.6, 177.4)
- removed the REF** at (288.6, 189.4)
- removed the REF** at (304.6, 195.4)
- removed the REF** at (288.6, 183.4)
- removed the REF** at (288.6, 195.4)
- added REF**: MountingHole_3.2mm_M3, MountingHole:MountingHole_3.2mm_M3, F.Cu at (304.6, 171.6)
- added REF**: MountingHole_3.2mm_M3, MountingHole:MountingHole_3.2mm_M3, F.Cu at (304.6, 178.9)
- added REF**: MountingHole_3.2mm_M3, MountingHole:MountingHole_3.2mm_M3, F.Cu at (288.6, 171.6)
- added REF**: MountingHole_3.2mm_M3, MountingHole:MountingHole_3.2mm_M3, F.Cu at (288.6, 178.9)
- added REF**: MountingHole_3.2mm_M3, MountingHole:MountingHole_3.2mm_M3, F.Cu at (288.6, 193.5)
- added REF**: MountingHole_3.2mm_M3, MountingHole:MountingHole_3.2mm_M3, F.Cu at (304.6, 193.5)
- added REF**: MountingHole_3.2mm_M3, MountingHole:MountingHole_3.2mm_M3, F.Cu at (288.6, 186.2)
- added REF**: MountingHole_3.2mm_M3, MountingHole:MountingHole_3.2mm_M3, F.Cu at (304.6, 186.2)
- J1: value Conn_01x08_Socket -> Conn_01x11_Socket; footprint Connector_PinHeader_2.54mm:PinHeader_1x08_P2.54mm_Vertical -> Connector_PinHeader_2.54mm:PinHeader_1x11_P2.54mm_Vertical
- J4: footprint Connector_JST:JST_XH_S2B-XH-A_1x02_P2.50mm_Horizontal -> Connector_JST:JST_XH_B2B-XH-A_1x02_P2.50mm_Vertical
- moved J1 17.4 mm to (309.4, 204.7)
- moved J4 5.77 mm to (303.9, 278.3)
Connections:
- A1 pad 19: SENSOR8 -> SENSOR1
- A1 pad 20: SENSOR7 -> SENSOR2
- A1 pad 21: SENSOR6 -> SENSOR3
- A1 pad 22: SENSOR5 -> SENSOR4
- A1 pad 23: SENSOR4 -> SENSOR5
- A1 pad 24: SENSOR3 -> SENSOR6
- A1 pad 25: SENSOR2 -> SENSOR7
- A1 pad 26: SENSOR1 -> SENSOR8
- J1 pad 1: SENSOR8 -> GND
- J1 pad 2: SENSOR7 -> 5V
- J1 pad 3: SENSOR6 -> LED_CTRL
- J1 pad 4: SENSOR5 -> SENSOR1
- J1 pad 5: SENSOR4 -> SENSOR2
- J1 pad 7: SENSOR2 -> SENSOR4
- J1 pad 8: SENSOR1 -> SENSOR5
Routing:
- net SENSOR8: track 5.26 -> 0.00 mm
- net SENSOR3: track 5.21 -> 0.00 mm
- net SENSOR7: track 5.21 -> 0.00 mm
- net SENSOR6: track 5.21 -> 0.00 mm
- net SENSOR5: track 5.21 -> 0.00 mm
- net SENSOR4: track 5.21 -> 0.00 mm
- net SENSOR2: track 5.21 -> 0.00 mm
- net SENSOR1: track 5.21 -> 0.05 mm
- net 7.4V: track 14.9 -> 12.5 mm
Other:
- outline, holes or cut-outs redrawn

Commit message: Add relevant sensor reading functions
Routing:
- net SENSOR7: track 0.00 -> 23.8 mm
- net SENSOR6: track 0.00 -> 23.8 mm
- net SENSOR5: track 0.00 -> 23.8 mm
- net SENSOR4: track 0.00 -> 23.8 mm
- net SENSOR3: track 0.00 -> 23.8 mm
- net SENSOR2: track 0.00 -> 23.8 mm
- net SENSOR8: track 0.00 -> 23.8 mm
- net SENSOR1: track 0.05 -> 23.8 mm
- net LED_CTRL: track 41.6 -> 62.5 mm
- net 5V: track 164.7 -> 185.2 mm
Other:
- board text removed: "Uyeristic Whip LF 11.30.2024"
Changed lines of the file:
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@@
 		)
 		(fp_text user "${REFERENCE}"
-			(at 7.27 3.81 360)
+			(at 7.27 3.81 0)
 			(layer "F.Fab")
 			(effects
@@
 		)
 		(fp_text user "${REFERENCE}"
-			(at 0 12.7 360)
+			(at 0 12.7 0)
 			(layer "F.Fab")
 			(effects
@@
 		)
 		(property "Value" "Arduino_Nano_v3.x"
-			(at 8.89 19.05 360)
+			(at 8.89 19.05 0)
 			(layer "F.Fab")
 			(effects
@@
 		)
 		(fp_text user "${REFERENCE}"
-			(at 6.35 19.05 360)
+			(at 6.35 19.05 0)
 			(layer "F.Fab")
 			(effects
@@
 		(layer "Edge.Cuts")
 	)
-	(gr_text "Uyeristic Whip\nLF 11.30.2024"
-		(at 296.59 216.07 0)
-		(layer "B.Cu")
-		(effects
-			(font
-				(size 1.7 1.7)
-				(thickness 0.3)
-				(bold yes)
-			)
-			(justify bottom mirror)
-		)
-	)
 	(gr_text "N20 Motor"
 		(at 250.45 267.45 0)
@@
 	)
 	(segment
+		(start 283.95 204.7)
+		(end 283.95 204.65)
+		(width 0.508)
+		(layer "B.Cu")
+		(net 5)
+	)
+	(segment
+		(start 287.81 226.82)
+		(end 287.81 208.56)
+		(width 0.508)
+		(layer "B.Cu")
+		(net 5)
+	)
+	(segment
+		(start 287.81 208.56)
+		(end 283.95 204.7)
+		(width 0.508)
+		(layer "B.Cu")
+		(net 5)
+	)
+	(segment
 		(start 300.51 242.06)
 		(end 297.87 244.7)
@@
 	)
 	(segment
+		(start 290.35 226.82)
+		(end 290.35 208.51)
+		(width 0.508)
+		(layer "B.Cu")
+		(net 7)
+	)
+	(segment
+		(start 290.35 208.51)
+		(end 286.49 204.65)
+		(width 0.508)
+		(layer "B.Cu")
+		(net 7)
+	)
+	(segment
 		(start 290.35 246.795)
 		(end 287.845 249.3)
@@
 	)
 	(segment
+		(start 297.97 226.82)
+		(end 297.97 208.51)
+		(width 0.508)
+		(layer "B.Cu")
+		(net 10)
+	)
+	(segment
+		(start 297.97 208.51)
+		(end 294.11 204.65)
+		(width 0.508)
+		(layer "B.Cu")
+		(net 10)
+	)
+	(segment
+		(start 300.51 208.51)
+		(end 296.65 204.65)
+		(width 0.508)
+		(layer "B.Cu")
+		(net 12)
+	)
+	(segment
+		(start 300.51 226.82)
+		(end 300.51 208.51)
+		(width 0.508)
+		(layer "B.Cu")
+		(net 12)
+	)
+	(segment
+		(start 305.59 208.51)
+		(end 301.73 204.65)
+		(width 0.508)
+		(layer "B.Cu")
+		(net 13)
+	)
+	(segment
 		(start 305.625 226.785)
 		(end 305.59 226.82)
@@
 	)
 	(segment
-		(start 303.05 242.06)
-		(end 298.91 246.2)
+		(start 305.59 226.82)
+		(end 305.59 208.51)
 		(width 0.508)
 		(layer "B.Cu")
-		(net 19)
+		(net 13)
 	)
 	(segment
-		(start 296.025 246.2)
-		(end 292.925 249.3)
+		(start 295.43 226.82)
+		(end 295.43 208.51)
 		(width 0.508)
 		(layer "B.Cu")
-		(net 19)
+		(net 16)
 	)
 	(segment
-		(start 298.91 246.2)
-		(end 296.025 246.2)
+		(start 295.43 208.51)
+		(end 291.57 204.65)
+		(width 0.508)
+		(layer "B.Cu")
+		(net 16)
+	)
+	(segment
+		(start 292.89 208.51)
+		(end 289.03 204.65)
+		(width 0.508)
+		(layer "B.Cu")
+		(net 17)
+	)
+	(segment
+		(start 292.89 226.82)
+		(end 292.89 208.51)
+		(width 0.508)
+		(layer "B.Cu")
+		(net 17)
+	)
+	(segment
+		(start 303.05 242.06)
+		(end 298.91 246.2)
 		(width 0.508)
 		(layer "B.Cu")
@@
 	)
 	(segment
-		(start 273.125 228.95)
-		(end 283.14 228.95)
+		(start 296.025 246.2)
+		(end 292.925 249.3)
 		(width 0.508)
 		(layer "B.Cu")
-		(net 22)
+		(net 19)
 	)
 	(segment
-		(start 290.385 264.54)
-		(end 290.385 264.535)
+		(start 298.91 246.2)
+		(end 296.025 246.2)
 		(width 0.508)
 		(layer "B.Cu")
-		(net 22)
+		(net 19)
 	)
 	(segment
@@
 	)
 	(segment
-		(start 315.465 221.525)
-		(end 315.45 221.54)
+		(start 273.125 228.95)
+		(end 283.14 228.95)
 		(width 0.508)
 		(layer "B.Cu")
@@
 	)
 	(segment
-		(start 315.45 227.575)
-		(end 313.95 229.075)
+		(start 306.81 206.34)
+		(end 310.61 210.14)
 		(width 0.508)
 		(layer "B.Cu")
@@
 	)
 	(segment
-		(start 295.465 249.86)
-		(end 293.975 251.35)
+		(start 290.385 264.54)
+		(end 290.385 264.535)
 		(width 0.508)
 		(layer "B.Cu")
@@
 	)
 	(segment
-		(start 315.45 221.54)
-		(end 315.45 227.575)
+		(start 295.465 249.86)
+		(end 293.975 251.35)
 		(width 0.508)
 		(layer "B.Cu")
@@
 	)
 	(segment
+		(start 310.61 210.14)
+		(end 310.61 218.75)
+		(width 0.508)
+		(layer "B.Cu")
+		(net 22)
+	)
+	(segment
 		(start 277.375 251.525)
 		(end 257.9 251.525)
@@
 	)
 	(segment
+		(start 315.45 227.575)
+		(end 313.95 229.075)
+		(width 0.508)
+		(layer "B.Cu")
+		(net 22)
+	)
+	(segment
 		(start 290.385 264.535)
 		(end 277.375 251.525)
@@
 	)
 	(segment
-		(start 313.95 229.075)
-		(end 287.525 229.075)
+		(start 306.81 204.65)
+		(end 306.81 206.34)
 		(width 0.508)
 		(layer "B.Cu")
@@
 	)
 	(segment
+		(start 310.61 218.75)
+		(end 315.45 223.59)
+		(width 0.508)
+		(layer "B.Cu")
+		(net 22)
+	)
+	(segment
+		(start 313.95 229.075)
+		(end 287.525 229.075)
+		(width 0.508)
+		(layer "B.Cu")
+		(net 22)
+	)
+	(segment
+		(start 315.45 223.59)
+		(end 315.45 227.575)
+		(width 0.508)
+		(layer "B.Cu")
+		(net 22)
+	)
+	(segment
 		(start 280.4 244.95)
 		(end 276.45 244.95)
@@
 	)
 	(segment
-		(start 309.335 218.475)
-		(end 314.875 218.475)
+		(start 314.825 230.9)
+		(end 309.13 230.9)
 		(width 0.508)
 		(layer "B.Cu")
@@
 	)
 	(segment
-		(start 317.5 228.225)
-		(end 314.825 230.9)
+		(start 313.65 204.23)
+		(end 313.65 218.9)
 		(width 0.508)
 		(layer "B.Cu")
@@
 	)
 	(segment
-		(start 317.5 221.1)
+		(start 317.5 222.75)
 		(end 317.5 228.225)
 		(width 0.508)
@@
 	)
 	(segment
-		(start 314.875 218.475)
-		(end 317.5 221.1)
+		(start 317.5 228.225)
+		(end 314.825 230.9)
 		(width 0.508)
 		(layer "B.Cu")
@@
 	)
 	(segment
-		(start 314.825 230.9)
-		(end 309.13 230.9)
+		(start 307.17 201.75)
+		(end 311.17 201.75)
 		(width 0.508)
 		(layer "B.Cu")
@@
 	)
 	(segment
+		(start 304.27 204.65)
+		(end 307.17 201.75)
+		(width 0.508)
+		(layer "B.Cu")
+		(net 24)
+	)
+	(segment
+		(start 311.17 201.75)
+		(end 313.65 204.23)
+		(width 0.508)
+		(layer "B.Cu")
+		(net 24)
+	)
+	(segment
+		(start 313.65 218.9)
+		(end 317.5 222.75)
+		(width 0.508)
+		(layer "B.Cu")
+		(net 24)
+	)
+	(segment
+		(start 303.05 208.51)
+		(end 299.19 204.65)
+		(width 0.508)
+		(layer "B.Cu")
+		(net 25)
+	)
+	(segment
+		(start 303.05 226.82)
+		(end 303.05 208.51)
+		(width 0.508)
+		(layer "B.Cu")
+		(net 25)
+	)
+	(segment

Commit message: Update Chassis PCB Design
Parts:
- moved REF** 0.11 mm to (304.6, 171.7)
- moved REF** 0.11 mm to (288.6, 171.7)
- moved REF** 0.06 mm to (304.6, 178.9)

Commit message: Finalize PCB Design and 3D Models
Parts:
- moved REF** 2.00 mm to (317.7, 258.4)
- moved REF** 2.00 mm to (275.7, 258.4)
- moved REF** 1.00 mm to (317.7, 276.2)
- moved REF** 1.00 mm to (275.7, 276.2)
Routing:
- removed copper zone on F.Cu, net GND
